File: robocrob/robocrob.kicad_pcb (KiCad board)
At the start: 2 copper layers, 77.3 x 57.3 mm, 6 parts, among them J1 Conn_01x03_Female, SW2 SW_DIP_x02

Commit message: ship it or die trying
Parts:
- removed SW2: SW_DIP_x02, Button_Switch_SMD:SW_DPDT_CK_JS202011JCQN
- added R1: 50, Resistor_SMD:R_1206_3216Metric_Pad1.42x1.75mm_HandSolder, B.Cu at (37.8, 38.6)
- added REF**: MountingHole_2.1mm, MountingHole:MountingHole_2.1mm, F.Cu at (27.9, 21.0)
- added REF**: MountingHole_2.1mm, MountingHole:MountingHole_2.1mm, F.Cu at (69.2, 17.8)
- added SW1: SW_DIP_x01, Button_Switch_SMD:SW_DIP_SPSTx01_Slide_6.7x4.1mm_W8.61mm_P2.54mm_LowProfile, B.Cu at (19.7, 40.0)
- J1: value Conn_01x03_Female -> Conn_01x02_Female; footprint Connector_PinHeader_2.54mm:PinHeader_1x03_P2.54mm_Vertical -> Connector_PinSocket_2.54mm:PinSocket_1x02_P2.54mm_Vertical
- moved J1 5.08 mm to (19.1, 28.6), turned to 180 degrees
Connections:
- DLEFT1 pad 1: GND -> Net-(DLEFT1-Pad1)
- DRIGHT1 pad 1: GND -> Net-(DLEFT1-Pad1)
- DRIGHT1 pad 2: Net-(DRIGHT1-Pad2) -> Net-(DLEFT1-Pad2)
- J1 pad 1: Net-(DLEFT1-Pad2) -> GND
- J1 pad 2: Net-(DRIGHT1-Pad2) -> Net-(DLEFT1-Pad2)
Routing:
- net Net-(DRIGHT1-Pad2): track 75.2 -> 0.00 mm
- net Net-(DLEFT1-Pad1): track 0.00 -> 37.9 mm
- net Net-(DLEFT1-Pad2): track 51.6 -> 68.4 mm
- net Net-(BT1-Pad1): track 13.2 -> 10.6 mm
Other:
- board size 77.3 x 57.3 mm -> 77.3 x 57.8 mm
- net class Default: trace_width 0.55 -> 0.85
- board text added: "+"
- board text added: "-"
- board text added: "3.3V Coin Cell Battery"
- board text added: "3v3"
- board text added: "American Crow - Corvus Brachyrhynchos From beak to tail, an American crow measures 40–50 cm (16–20 in), almost half of which is tail. Mass varies from about 300 to 600 g (11 to 21 oz). The most usual call is CAWW!-CAWW!-CAWW! The American crow is one of only a few species of bird that has been observed modifying and using tools to obtain food."
- board text added: "Merry Christmas! Chris Johnston 2020"
- board text added: "_"
- board text removed: "Chris Johnston CSS Secret Santa 2020"
- board text removed: "Left Eye 3v3"
- board text removed: "Right Eye 3v3"
